File: Hardware/ESP_Programmer/ESP_Programmer.kicad_sch (KiCad schematic)
At the start: 9 parts, among them J1 Conn_01x05_Pin, J2 USB_OTG, SW10 SW_MEC_5E, SW9 SW_MEC_5E, U2 CH340G

Commit message: Terminado el programador de ESp
Parts:
- removed U2: CH340G, Package_SO:SOIC-16_3.9x9.9mm_P1.27mm, symbol Interface_USB:CH340G
- added C11: 10uF, Capacitor_SMD:CP_Elec_4x5.4, symbol Device:C_Polarized_Small
- added C12: 22uF, Capacitor_SMD:CP_Elec_4x5.4, symbol Device:C_Polarized_Small
- added C13, C14: 1uF, Capacitor_SMD:C_0603_1608Metric, symbol Device:C
- added D1, D2: LED, LED_SMD:LED_0603_1608Metric_Pad1.05x0.95mm_HandSolder, symbol Device:LED
- added R1, R2: 221, Resistor_SMD:R_0603_1608Metric, symbol Device:R_US
- added U1: CH340C, Package_SO:SOIC-16_3.9x9.9mm_P1.27mm, symbol Interface_USB:CH340C
- added U3: AMS1117-3.3, Package_TO_SOT_SMD:SOT-223-3_TabPin2, symbol Regulator_Linear:AMS1117-3.3
- R8, R9: footprint https://ar.mouser.com/datasheet/2/447/PYu_RT_1_to_0_01_RoHS_L_15-3461507.pdf -> Resistor_SMD:R_0603_1608Metric
Connections:
- net +5V: now also C11.1, C13.1, U3.3 (VI); no longer C2.1
- net GND: now also C11.2, C12.2, C13.2, C14.2, U1.1 (GND), U3.1 (GND)
- net at C1.2: now also U1.4 (V3)
- net at J2.2 (D-): now also U1.6 (UD-)
- net at J2.3 (D+): now also U1.5 (UD+)
- net Tx: now reaches J1.5 (Pin_5)
- net Tx: now also D1.1 (K), U1.2 (TXD)
- net Rx: now reaches J1.4 (Pin_4)
- net Rx: now also D2.1 (K), U1.3 (RXD)
- new net: D1.2 (A), R1.2
- new net: D2.2 (A), R2.2
- new net +3.3V: C12.1, C14.1, C2.1, R1.1, R2.1, U1.16 (VCC), U3.2 (VO)
- no-connect marks 9 -> 7
