File: Hardware/Cnv-Inv-Micro/MedicionCorriente.kicad_sch (KiCad schematic)
At the start: 5 parts, among them U15 ACS712xLCTR-05B

Commit message: Avances en PCB conversor y inversor - Simulaciones de modulacion
Parts:
- renumbered C23 to C12, C24 to C13, D16 to D10, R39 to R27, U15 to U11
Changed lines of the file:
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@@
 		(dnp no)
 		(fields_autoplaced yes)
-		(property "Reference" "C24"
+		(property "Reference" "C13"
 			(at 180.34 100.3299 0)
 			(effects
@@
 			(project "VFD_V1"
 				(path "/e60c11d9-ab9e-4760-a4a7-008fcec65a72/c6551446-5e26-4d9a-a5bc-1c867d865e21/5d7c7860-569e-4893-a242-75c72190872b"
-					(reference "C24")
+					(reference "C13")
 					(unit 1)
 				)
@@
 		(on_board yes)
 		(dnp no)
-		(property "Reference" "#PWR050"
+		(property "Reference" "#PWR035"
 			(at 115.57 118.11 0)
 			(effects
@@
 			(project "VFD_V1"
 				(path "/e60c11d9-ab9e-4760-a4a7-008fcec65a72/c6551446-5e26-4d9a-a5bc-1c867d865e21/5d7c7860-569e-4893-a242-75c72190872b"
-					(reference "#PWR050")
+					(reference "#PWR035")
 					(unit 1)
 				)
@@
 		(dnp no)
 		(fields_autoplaced yes)
-		(property "Reference" "D16"
+		(property "Reference" "D10"
 			(at 144.78 105.4099 90)
 			(effects
@@
 			(project ""
 				(path "/e60c11d9-ab9e-4760-a4a7-008fcec65a72/c6551446-5e26-4d9a-a5bc-1c867d865e21/5d7c7860-569e-4893-a242-75c72190872b"
-					(reference "D16")
+					(reference "D10")
 					(unit 1)
 				)
@@
 		(on_board yes)
 		(dnp no)
-		(property "Reference" "#PWR053"
+		(property "Reference" "#PWR038"
 			(at 176.53 114.3 0)
 			(effects
@@
 			(project "VFD_V1"
 				(path "/e60c11d9-ab9e-4760-a4a7-008fcec65a72/c6551446-5e26-4d9a-a5bc-1c867d865e21/5d7c7860-569e-4893-a242-75c72190872b"
-					(reference "#PWR053")
+					(reference "#PWR038")
 					(unit 1)
 				)
@@
 		(dnp no)
 		(fields_autoplaced yes)
-		(property "Reference" "C23"
+		(property "Reference" "C12"
 			(at 133.35 106.6799 0)
 			(effects
@@
 			(project ""
 				(path "/e60c11d9-ab9e-4760-a4a7-008fcec65a72/c6551446-5e26-4d9a-a5bc-1c867d865e21/5d7c7860-569e-4893-a242-75c72190872b"
-					(reference "C23")
+					(reference "C12")
 					(unit 1)
 				)
@@
 		(on_board yes)
 		(dnp no)
-		(property "Reference" "#PWR051"
+		(property "Reference" "#PWR036"
 			(at 129.54 119.38 0)
 			(effects
@@
 			(project "VFD_V1"
 				(path "/e60c11d9-ab9e-4760-a4a7-008fcec65a72/c6551446-5e26-4d9a-a5bc-1c867d865e21/5d7c7860-569e-4893-a242-75c72190872b"
-					(reference "#PWR051")
+					(reference "#PWR036")
 					(unit 1)
 				)
@@
 		(dnp no)
 		(fields_autoplaced yes)
-		(property "Reference" "R39"
+		(property "Reference" "R27"
 			(at 134.62 93.98 90)
 			(effects
@@
 			(project "VFD_V1"
 				(path "/e60c11d9-ab9e-4760-a4a7-008fcec65a72/c6551446-5e26-4d9a-a5bc-1c867d865e21/5d7c7860-569e-4893-a242-75c72190872b"
-					(reference "R39")
+					(reference "R27")
 					(unit 1)
 				)
@@
 		(on_board yes)
 		(dnp no)
-		(property "Reference" "#PWR052"
+		(property "Reference" "#PWR037"
 			(at 142.24 118.11 0)
 			(effects
@@
 			(project "VFD_V1"
 				(path "/e60c11d9-ab9e-4760-a4a7-008fcec65a72/c6551446-5e26-4d9a-a5bc-1c867d865e21/5d7c7860-569e-4893-a242-75c72190872b"
-					(reference "#PWR052")
+					(reference "#PWR037")
 					(unit 1)
 				)
@@
 		(dnp no)
 		(fields_autoplaced yes)
-		(property "Reference" "U15"
+		(property "Reference" "U11"
 			(at 117.7133 87.63 0)
 			(effects
@@
 			(project ""
 				(path "/e60c11d9-ab9e-4760-a4a7-008fcec65a72/c6551446-5e26-4d9a-a5bc-1c867d865e21/5d7c7860-569e-4893-a242-75c72190872b"
-					(reference "U15")
-					(unit 1)
-				)
+					(reference "U11")
+					(unit 1)
+				)
