File: Hardware/Cnv-Inv-Micro/ModuloConmutadorPushpull.kicad_sch (KiCad schematic)
At the start: 1 part

Commit message: Avances en PCB conversor y inversor - Simulaciones de modulacion
Parts:
- renumbered R34 to R22
Changed lines of the file:
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@@
 		(dnp no)
 		(fields_autoplaced yes)
-		(property "Reference" "R34"
+		(property "Reference" "R22"
 			(at 104.14 86.36 90)
 			(effects
@@
 			(project "VFD_V1"
 				(path "/e60c11d9-ab9e-4760-a4a7-008fcec65a72/c6551446-5e26-4d9a-a5bc-1c867d865e21/114be0da-6ec0-43cc-95ec-fead423de7f2"
-					(reference "R34")
+					(reference "R22")
 					(unit 1)
 				)
 				(path "/e60c11d9-ab9e-4760-a4a7-008fcec65a72/c6551446-5e26-4d9a-a5bc-1c867d865e21/4ead1ef3-6642-476a-91a4-2f6f295e53fc"
-					(reference "R36")
+					(reference "R24")
 					(unit 1)
 				)
