File: Hardware/Cnv-Inv-Micro/SistemaControlConversor.kicad_sch (KiCad schematic)
At the start: 12 parts, among them U16 TL494

Commit message: Avances en PCB conversor y inversor - Simulaciones de modulacion
Parts:
- renumbered C25 to C14, C26 to C15, C27 to C16, R40 to R28, R41 to R29, R42 to R30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
Connections:
- net Gnd: now also R32.1, R33.1
- net Out_Signal_A: now also R32.2, U12.9 (E1); no longer R32.1
- net Out_Signal_B: now also R33.2, U12.10 (E2); no longer R33.1
Other:
- moved on the sheet: R32, R33
