File: Hardware/Cnv-Inv-Micro/VFD_V1.kicad_pcb (KiCad board)
At the start: 2 copper layers, 256.6 x 180.1 mm, 209 parts, among them J1 Conn_01x03, J2 Screw_Terminal_01x07, J3 Screw_Terminal_01x03, Q1 TK8A65D, Q10 SS8050, Q11 SS8050, Q12 SS8050, Q13 SS8050, Q14 SS8550, Q15 IRFB4110PBF, Q16 SS8050, Q17 SS8550, Q18 IRFB4110PBF, Q19 SS8050, Q2 TK8A65D, Q20 SS8550, Q21 IRFB4110PBF, Q22 SS8050, Q23 SS8550, Q24 IRFB4110PBF, Q3 TK8A65D, Q4 TK8A65D, Q5 TK8A65D, Q6 TK8A65D, Q7 SS8050, Q8 SS8050, Q9 SS8050, SW1 SW_MEC_5E, U1 TMA-1205S-2WR2, U10 6N135, U11 IR2104, U12 6N135, U13 6N135, U14 IR2104, U15 ACS712xLCTR-05B, U16 TL494, U17 TL431PK, U18 PC817, U19 PC817, U2 TMA-1205S-2WR2, U20 TL431PK, U21 PC817, U22 PC817, U23 PC817, U3 AMS1117-3.3, U4 STM32F103C8Tx, U5 TMA-12012S-2WR3, U6 6N135, U7 6N135, U8 IR2104, U9 6N135, Y1 Crystal 8MHz

Commit message: Normalizacion placa micros
Parts:
- moved U2 41.3 mm to (39.0, 94.2)
Connections:
- net SW_Gnd renamed Gnd_Micro
Routing:
- net Gnd_Micro: track 209.3 -> 177.3 mm, vias 2 -> 6
- net Reset: track 26.7 -> 30.9 mm, vias 0 -> 1
- net (no net): track 0.00 -> 2.85 mm, vias 0 -> 1
- added copper zone on B.Cu, net Gnd_Micro
- added copper zone on F.Cu, net Gnd_Micro

Commit message: Avances en PCB conversor y inversor - Simulaciones de modulacion
Parts:
- removed 12V_Pwr_In1, Emg_Button1: Screw_Terminal_01x02, TerminalBlock_Phoenix:TerminalBlock_Phoenix_MKDS-1,5-2_1x02_P5.00mm_Horizontal
- removed the C10 at (55.4, 121.9)
- removed the C11 at (78.2, 112.3)
- removed the C12 at (94.9, 114.2)
- removed the C13 at (57.2, 131.4)
- removed the C14 at (64.1, 131.4)
- removed the C15 at (26.3, 103.9)
- removed the C16 at (26.3, 129.9)
- removed the C4 at (18.4, 103.8)
- removed the C5 at (71.1, 128.9)
- removed the C6 at (73.4, 112.4)
- removed the C7 at (63.5, 124.1)
- removed the C8 at (18.1, 129.0)
- removed the C9 at (66.9, 113.4)
- removed Cnv_Control_A1, Cnv_Control_A2, HMI_Signal_B2: Conn_01x05, Connector_Molex:Molex_KK-254_AE-6410-05A_1x05_P2.54mm_Vertical
- removed Conv_PwrBus_A2, Inv_PwrBus_A1, Micro_PwrBus_A1, Micro_PwrBus_B1: Conn_01x02, Connector_Phoenix_MSTB:PhoenixContact_MSTBVA_2,5_2-G-5,08_1x02_P5.08mm_Vertical
- removed the D10 at (53.2, 135.5)
- removed D12: LED_Red, LED_SMD:LED_0603_1608Metric_Pad1.05x0.95mm_HandSolder
- removed D17: LED_Green, LED_THT:LED_Rectangular_W5.0mm_H2.0mm
- removed the D7 at (51.3, 120.6)
- removed HMI_Pwr_A1, Inv_Pwr_A1, TermoSwitch1: Conn_01x02, Connector_Molex:Molex_KK-254_AE-6410-02A_1x02_P2.54mm_Vertical
- removed Inv_Signal1_A1, Inv_Signal2_A1: Conn_01x04, Connector_Molex:Molex_KK-254_AE-6410-04A_1x04_P2.54mm_Vertical
- removed J1: Conn_01x03, Connector_PinHeader_2.54mm:PinHeader_1x03_P2.54mm_Vertical_SMD_Pin1Left
- removed J2: Screw_Terminal_01x07, TerminalBlock_Phoenix:TerminalBlock_Phoenix_PT-1,5-7-5.0-H_1x07_P5.00mm_Horizontal
- removed J3: Screw_Terminal_01x03, TerminalBlock_Phoenix:TerminalBlock_Phoenix_MKDS-1,5-3-5.08_1x03_P5.08mm_Horizontal
- removed J_Pw_In+1, J_Pw_In-1: Conn_01x02, BananaSocket_THT:BananaSocket - 2P - 4mm
- removed Motor_Out_B1: Conn_01x03, Connector_Phoenix_MC_HighVoltage:PhoenixContact_MCV_1,5_3-G-5.08_1x03_P5.08mm_Vertical
- removed Out_Motor1: Screw_Terminal_01x03, TerminalBlock_MetzConnect:TerminalBlock_MetzConnect_Type703_RT10N03HGLU_1x03_P9.52mm_Horizontal
- removed the R10 at (81.7, 127.3)
- removed the R11 at (81.7, 125.7)
- removed the R12 at (81.7, 124.2)
- removed the R13 at (81.7, 122.7)
- removed the R14 at (81.7, 121.2)
- removed the R3 at (66.9, 124.1)
- removed the R4 at (53.5, 119.0)
- removed the R5 at (69.6, 116.0)
- removed R53, R63, R65: 4.7k, Resistor_SMD:R_0603_1608Metric_Pad0.98x0.95mm_HandSolder
- removed R54, R64, R66: 3.3k, Resistor_SMD:R_0603_1608Metric_Pad0.98x0.95mm_HandSolder
- removed the R6 at (57.2, 135.5)
- removed R62: 1.2k, Resistor_SMD:R_0603_1608Metric_Pad0.98x0.95mm_HandSolder
- removed the R7 at (79.9, 117.6)
- removed the R8 at (79.9, 119.1)
- removed the R9 at (81.7, 128.8)
- removed SW1: SW_MEC_5E, TatilSwitch:Vertical SPST SMD Tactile Switches
- removed SWD_Program1: Conn_02x05_Odd_Even, Connector_IDC:IDC-Header_2x05_P2.54mm_Vertical_SMD
- removed U19, U22, U23: PC817, Package_DIP:DIP-4_W7.62mm_SMDSocket_SmallPads
- removed the U2 at (39.0, 94.2)
- removed the U3 at (86.0, 113.3)
- removed the U4 at (61.2, 117.6)
- removed the U5 at (28.1, 109.3)
- removed Y1: Crystal 8MHz, Crystal:Crystal_SMD_HC49-SD
- added 12V_Pwr1: Screw_Terminal_01x02, TerminalBlock_Phoenix:TerminalBlock_Phoenix_MKDS-1,5-2_1x02_P5.00mm_Horizontal, F.Cu at (335.3, 47.2)
- added C1: 4.7uF, Capacitor_SMD:CP_Elec_4x5.4, F.Cu at (102.1, 103.5)
- added C2: 4.7uF, Capacitor_SMD:CP_Elec_4x5.4, F.Cu at (68.7, 103.5)
- added Cnv_Pwr1: Conn_01x02, Connector_Molex:Molex_KK-254_AE-6410-02A_1x02_P2.54mm_Vertical, F.Cu at (341.2, 29.2)
- added Inv_Pwr1: Conn_01x02, Connector_Molex:Molex_KK-254_AE-6410-02A_1x02_P2.54mm_Vertical, F.Cu at (332.0, 29.2)
- added Inv_Pwr2: Conn_01x02, Connector_Molex:Molex_KK-254_AE-6410-02A_1x02_P2.54mm_Vertical, F.Cu at (350.0, 37.6)
- added Motor_Out2: Conn_01x03, Connector_Phoenix_MC_HighVoltage:PhoenixContact_MCV_1,5_3-G-5.08_1x03_P5.08mm_Vertical, F.Cu at (360.0, 28.8)
- added Motor_Pwr1: Screw_Terminal_01x03, TerminalBlock_Dinkle:TerminalBlock_Dinkle_DT-55-B01X-03_P10.00mm, F.Cu at (378.0, 51.2)
- added Pw_In+1: Conn_01x02, BananaSocket_THT:BananaSocket - 2P - 4mm, F.Cu at (343.5, 69.6)
- added Pw_In-1: Conn_01x02, BananaSocket_THT:BananaSocket - 2P - 4mm, F.Cu at (377.7, 69.6)
- added R48: 1.2k, Resistor_THT:R_Axial_DIN0207_L6.3mm_D2.5mm_P10.16mm_Horizontal, F.Cu at (339.6, 38.0)
- D11: value LED_Yellow -> LED_Green; footprint LED_SMD:LED_0603_1608Metric_Pad1.05x0.95mm_HandSolder -> LED_THT:LED_Rectangular_W5.0mm_H2.0mm
- U1: value TMA-1205S-2WR2 -> TMA-12012S-2WR3
- U2: renamed from U6; footprint Package_DIP:DIP-8_W7.62mm -> Package_SO:SOP-8_6.62x9.15mm_P2.54mm
- U3: renamed from U7; footprint Package_DIP:DIP-8_W7.62mm -> Package_SO:SOP-8_6.62x9.15mm_P2.54mm
- U5: renamed from U9; footprint Package_DIP:DIP-8_W7.62mm -> Package_SO:SOP-8_6.62x9.15mm_P2.54mm
- U6: renamed from U10; footprint Package_DIP:DIP-8_W7.62mm -> Package_SO:SOP-8_6.62x9.15mm_P2.54mm
- U8: renamed from U12; footprint Package_DIP:DIP-8_W7.62mm -> Package_SO:SOP-8_6.62x9.15mm_P2.54mm
- U9: renamed from U13; footprint Package_DIP:DIP-8_W7.62mm -> Package_SO:SOP-8_6.62x9.15mm_P2.54mm
- moved D11 265.9 mm to (335.2, 57.4)
- moved Cooler1 253.4 mm to (350.0, 29.2), turned to 180 degrees
- moved U1 76.0 mm to (95.9, 105.1), turned to -90 degrees
- moved TP6 61.4 mm to (188.7, 27.9)
- moved 12V_Inv1 34.9 mm to (111.1, 103.4)
- moved U8 25.6 mm to (90.9, 92.1)
- moved U9 25.6 mm to (103.1, 92.1)
- moved U5 25.5 mm to (66.6, 92.1)
- moved U3 25.5 mm to (53.9, 92.0)
- moved U2 25.5 mm to (41.9, 92.0)
- moved U6 25.4 mm to (79.0, 92.1)
- moved Q12 24.6 mm to (105.0, 74.3)
- moved C10 24.6 mm to (97.9, 82.3)
- moved C7 24.6 mm to (44.3, 74.3)
- moved D7 24.6 mm to (40.3, 73.1)
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- renumbered J_Pwr_12V_Inv_B1 to 12V_Inv1, Cnv_Pwr_12V_B1 to 12V_PwrCnv1, C21 to C10, C22 to C11, C23 to C12, C24 to C13, C25 to C14, C26 to C15, C27 to C16, C28 to C17, C29 to C18, C1 to C3, C2 to C4, C3 to C5, C17 to C6, C18 to C7, C19 to C8, C20 to C9, D16 to D10, D13 to D7, D14 to D8, D15 to D9, HVDCBus_B1 to HVDCBus1, J_Inv_Signal1_B1 to Inv_Signal1, J_Inv_Signal2_B1 to Inv_Signal2, J_Motor_Out_A1 to Motor_Out1, Pwr_In+_A1 to Pwr+1, Pwr_In+_B1 to Pwr+2, Pwr_In-_A1 to Pwr-1, Pwr_In-_B1 to Pwr-2, R22 to R10, R23 to R11, R24 to R12, R25 to R13, R26 to R14, R27 to R15, R28 to R16, R29 to R17, R30 to R18, R31 to R19, R32 to R20, R33 to R21, R34 to R22, R35 to R23, R36 to R24, R37 to R25, R38 to R26, R39 to R27, R40 to R28, R41 to R29, R15 to R3, R42 to R30, R43 to R31, R44 to R32, R45 to R33, R46 to R34, R47 to R35, R48 to R36, R49 to R37, R50 to R38, R51 to R39, R16 to R4, R52 to R40, R55 to R41, R56 to R42, R57 to R43, R58 to R44, R59 to R45, R60 to R46, R61 to R47, R17 to R5, R18 to R6, R19 to R7, R20 to R8, R21 to R9, TP9 to TP1, TP7 to TP2, TP8 to TP3, TP1 to TP4, TP4 to TP5, TP5 to TP6, TP6 to TP7, TP2 to TP8, TP3 to TP9, U14 to U10, U15 to U11, U16 to U12, U17 to U13, U18 to U14, U20 to U15, U21 to U16, U8 to U4, U11 to U7
Connections:
- 12V_Inv1 pad 1: GND_Inv -> Net-(12V_Inv1-Pin_1)
- 12V_Inv1 pad 2: /Inversor/12V_Inv -> Net-(12V_Inv1-Pin_2)
- Cooler1 pad 2: Out_Emg1 -> /Interfaz de conexión/Gnd_Cnv
- D11 pad 2: LED_State -> /Interfaz de conexión/12V_Cnv
- U1 pad 1: /Micro/12V_Cnv -> Net-(12V_Inv1-Pin_2)
- U1 pad 2: Gnd_Cnv -> Net-(12V_Inv1-Pin_1)
- U1 pad 4: Net-(HMI_Pwr_A1-Pin_2) -> GND_Inv
- U1 pad 6: Net-(HMI_Pwr_A1-Pin_1) -> /Inversor/12V_Inv
Routing:
- net Gnd_Micro: track 177.3 -> 0.00 mm, vias 6 -> 0
- net 3V3_Micro: track 152.8 -> 0.00 mm
- net GND_Cnv: track 287.1 -> 228.1 mm, vias 1 -> 20
- net /Interfaz de conexión/12V_Cnv: track 0.00 -> 40.6 mm
- net Net-(C4-Pad1): track 113.1 -> 80.1 mm, vias 0 -> 48
- net /Interfaz de conexión/Gnd_Cnv: track 0.00 -> 32.0 mm
- net Mid_V: track 66.6 -> 34.6 mm, vias 1 -> 16
- net Reset: track 30.9 -> 0.00 mm, vias 1 -> 0
- net SW_Clk: track 27.4 -> 0.00 mm
- net Net-(D11-K): track 1.86 -> 25.4 mm
- net Net-(12V_Inv1-Pin_1): track 0.00 -> 23.1 mm
- net Net-(Motor_Out2-Pin_3): track 0.00 -> 23.0 mm
- net Net-(D3-A2): track 49.0 -> 71.8 mm, vias 0 -> 9
- net SW_DIO: track 22.8 -> 0.00 mm
- net Net-(Motor_Out2-Pin_2): track 0.00 -> 21.0 mm
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- added copper zone on B.Cu, net (none)
- added copper zone on B.Cu, net /Inversor/Gnd_Micro
- added copper zone on F.Cu, net /Inversor/Gnd_Micro
- added copper zone on F.Cu, net GND_Cnv
- added copper zone on B.Cu, net GND_Inv
- added copper zone on F.Cu, net GND_Inv
- removed copper zone on B.Cu, net Gnd_Micro
- removed copper zone on F.Cu, net Gnd_Micro
Other:
- board size 256.6 x 180.1 mm -> 387.7 x 100.4 mm
- board text added: "12V"
- board text added: "Gnd"
