File: Hardware/Cnv-Inv-Micro/conversor.kicad_sch (KiCad schematic)
At the start: 31 parts

Commit message: Avances en PCB conversor y inversor - Simulaciones de modulacion
Parts:
- removed J_Pw_In+1, J_Pw_In-1: Conn_01x02, BananaSocket_THT:BananaSocket - 2P - 4mm, symbol Connector_Generic:Conn_01x02
- C3: renamed from C1; value C_Electrolitic -> 4700uF
- C4: renamed from C2; value C_Electrolitic -> 4700uF
- renumbered Cnv_Pwr_12V_B1 to 12V_PwrCnv1, C3 to C5, Pwr_In+_A1 to Pwr+1, Pwr_In+_B1 to Pwr+2, Pwr_In-_A1 to Pwr-1, Pwr_In-_B1 to Pwr-2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
Other:
- moved on the sheet: C3
