File: Hardware/HMI_LVDC-Inverter/INPUT_ISO_1.kicad_sch (KiCad schematic)
At the start: 3 parts, among them U11 4N25

Commit message: Terminada la placa del HMI con revisión de reglas de diseño
Parts:
- removed U11: 4N25, Package_DIP:DIP-6_W7.62mm_SMDSocket_SmallPads, symbol Isolator:4N25
- added U17: PC817, Package_DIP:DIP-4_W7.62mm_SMDSocket_SmallPads, symbol Isolator:PC817
Connections:
- net GND: now also U17.3
- net INPUT: now also U17.4
- net INPUT_ISO: now also U17.2
- net at R36.1: now also U17.1
Other:
- moved on the sheet: R35
Changed lines of the file:
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@@
 	)
 	(junction
-		(at 133.35 87.63)
+		(at 133.35 85.09)
 		(diameter 0)
 		(color 0 0 0 0)
@@
 	(wire
 		(pts
-			(xy 133.35 87.63) (xy 134.62 87.63)
+			(xy 133.35 85.09) (xy 134.62 85.09)
 		)
 		(stroke
@@
 	(wire
 		(pts
-			(xy 133.35 77.47) (xy 133.35 78.74)
-		)
-		(stroke
-			(width 0)
-			(type default)
-		)
-	)
-	(wire
-		(pts
-			(xy 132.08 87.63) (xy 133.35 87.63)
+			(xy 133.35 74.93) (xy 133.35 76.2)
+		)
+		(stroke
+			(width 0)
+			(type default)
+		)
+	)
+	(wire
+		(pts
+			(xy 132.08 85.09) (xy 133.35 85.09)
 		)
 		(stroke
@@
 	(wire
 		(pts
-			(xy 133.35 86.36) (xy 133.35 87.63)
-		)
-		(stroke
-			(width 0)
-			(type default)
-		)
-	)
-	(wire
-		(pts
-			(xy 132.08 77.47) (xy 133.35 77.47)
+			(xy 133.35 83.82) (xy 133.35 85.09)
+		)
+		(stroke
+			(width 0)
+			(type default)
+		)
+	)
+	(wire
+		(pts
+			(xy 132.08 74.93) (xy 133.35 74.93)
 		)
 		(stroke
@@
 	(global_label "+3.3V_ESP"
 		(shape input)
-		(at 132.08 77.47 180)
+		(at 132.08 74.93 180)
 		(fields_autoplaced yes)
 		(effects
@@
 		)
 		(property "Intersheetrefs" "${INTERSHEET_REFS}"
-			(at 123.41 77.47 0)
+			(at 123.41 74.93 0)
 			(effects
 				(font
@@
 	(hierarchical_label "INPUT"
 		(shape bidirectional)
-		(at 132.08 87.63 180)
+		(at 132.08 85.09 180)
 		(effects
 			(font
@@
 	(symbol
 		(lib_id "Device:R_US")
-		(at 133.35 82.55 180)
+		(at 133.35 80.01 180)
 		(unit 1)
 		(exclude_from_sim no)
@@
 		(dnp no)
 		(property "Reference" "R35"
-			(at 126.746 81.788 0)
+			(at 126.746 79.248 0)
 			(effects
 				(font
@@
 		)
 		(property "Value" "33.2K"
-			(at 125.984 83.566 0)
+			(at 125.984 81.026 0)
 			(effects
 				(font
@@
 		)
 		(property "Footprint" "Resistor_SMD:R_0603_1608Metric_Pad0.98x0.95mm_HandSolder"
-			(at 132.334 82.296 90)
+			(at 132.334 79.756 90)
 			(effects
 				(font
@@
 		)
 		(property "Datasheet" "https://www.lcsc.com/datasheet/C706161.pdf"
-			(at 133.35 82.55 0)
+			(at 133.35 80.01 0)
 			(effects
 				(font
@@
 		)
 		(property "Description" "Resistor, US symbol"
-			(at 133.35 82.55 0)
+			(at 133.35 80.01 0)
 			(effects
 				(font
@@
 		)
 		(property "Footprint checked" "Yes"
-			(at 133.35 82.55 0)
+			(at 133.35 80.01 0)
 			(effects
 				(font
@@
 		)
 		(property "Symbol checked" "Yes"
-			(at 133.35 82.55 0)
+			(at 133.35 80.01 0)
 			(effects
 				(font
@@
 		)
 		(property "Price" "0.0095"
-			(at 133.35 82.55 0)
+			(at 133.35 80.01 0)
 			(effects
 				(font
@@
 		)
 		(property "Footprint Checked" ""
-			(at 133.35 82.55 0)
+			(at 133.35 80.01 0)
 			(effects
 				(font
@@
 		)
 		(property "Compra" "https://www.lcsc.com/product-detail/C706161.html"
-			(at 133.35 82.55 0)
+			(at 133.35 80.01 0)
 			(effects
 				(font
@@
 		)
 		(property "Manufacturer" "YAGEO"
-			(at 133.35 82.55 0)
+			(at 133.35 80.01 0)
 			(effects
 				(font
@@
 		)
 		(property "Sim.Library" ""
-			(at 133.35 82.55 0)
+			(at 133.35 80.01 0)
 			(effects
 				(font
@@
 	)
 	(symbol
-		(lib_id "Isolator:4N25")
+		(lib_id "Isolator:PC817")
 		(at 142.24 87.63 0)
 		(mirror y)
@@
 		(on_board yes)
 		(dnp no)
-		(property "Reference" "U11"
-			(at 141.986 80.01 0)
-			(effects
-				(font
-					(size 1.27 1.27)
-				)
-			)
-		)
-		(property "Value" "4N25"
-			(at 141.986 82.042 0)
-			(effects
-				(font
-					(size 1.27 1.27)
-				)
-			)
-		)
-		(property "Footprint" "Package_DIP:DIP-6_W7.62mm_SMDSocket_SmallPads"
+		(fields_autoplaced yes)
+		(property "Reference" "U17"
+			(at 142.24 78.74 0)
+			(effects
+				(font
+					(size 1.27 1.27)
+				)
+			)
+		)
+		(property "Value" "PC817"
+			(at 142.24 81.28 0)
+			(effects
+				(font
+					(size 1.27 1.27)
+				)
+			)
+		)
+		(property "Footprint" "Package_DIP:DIP-4_W7.62mm_SMDSocket_SmallPads"
 			(at 147.32 92.71 0)
 			(effects
@@
 			)
 		)
-		(property "Datasheet" "https://www.lcsc.com/datasheet/C898941.pdf"
+		(property "Datasheet" "https://www.lcsc.com/datasheet/C3008368.pdf"
 			(at 142.24 87.63 0)
 			(effects
@@
 			)
 		)
-		(property "Description" "DC Optocoupler Base Connected, Vce 30V, CTR 20%, Viso 2500V, DIP6"
+		(property "Description" "DC Optocoupler, Vce 35V, CTR 50-300%, DIP-4"
 			(at 142.24 87.63 0)
 			(effects
@@
 			)
 		)
-		(property "Compra" "https://www.lcsc.com/product-detail/C898941.html?s_z=n_4N25%2520SMD-6P"
+		(property "Compra" "https://www.lcsc.com/product-detail/C3008368.html"
 			(at 142.24 87.63 0)
 			(effects
@@
 			)
 		)
-		(property "Manufacturer" "onsemi"
+		(property "Manufacturer" "UMW"
 			(at 142.24 87.63 0)
 			(effects
@@
 			)
 		)
-		(property "Price" "0.9182"
+		(property "Price" "0.0347"
 			(at 142.24 87.63 0)
 			(effects
@@
 			)
 		)
+		(pin "2"
+		)
+		(pin "3"
+		)
+		(pin "4"
+		)
 		(pin "1"
-		)
-		(pin "3"
-		)
-		(pin "4"
-		)
-		(pin "6"
-		)
-		(pin "2"
-		)
-		(pin "5"
 		)
 		(instances
 			(project "HMI_LVDC-Inverter"
 				(path "/0057333c-5edf-4047-9690-4d1b87a98977/e510606f-6f04-4711-9f2b-d43d4de4a4de/055a40fe-cd38-468e-af40-51b3396e74eb"
-					(reference "U14")
+					(reference "U20")
 					(unit 1)
 				)
 				(path "/0057333c-5edf-4047-9690-4d1b87a98977/e510606f-6f04-4711-9f2b-d43d4de4a4de/56ca9b1f-7ac9-4571-b846-7d181a59aeeb"
-					(reference "U12")
+					(reference "U18")
 					(unit 1)
 				)
 				(path "/0057333c-5edf-4047-9690-4d1b87a98977/e510606f-6f04-4711-9f2b-d43d4de4a4de/6a364d1f-798c-4d3f-8ad2-c49dde5e0a04"
-					(reference "U16")
+					(reference "U22")
 					(unit 1)
 				)
 				(path "/0057333c-5edf-4047-9690-4d1b87a98977/e510606f-6f04-4711-9f2b-d43d4de4a4de/8ed63270-0053-4d5b-bff7-f9f37411008b"
-					(reference "U13")
+					(reference "U19")
 					(unit 1)
 				)
 				(path "/0057333c-5edf-4047-9690-4d1b87a98977/e510606f-6f04-4711-9f2b-d43d4de4a4de/bd0135dc-8da7-4e5d-91da-103a4a8ec09c"
-					(reference "U11")
+					(reference "U17")
 					(unit 1)
 				)
 				(path "/0057333c-5edf-4047-9690-4d1b87a98977/e510606f-6f04-4711-9f2b-d43d4de4a4de/d5a41d21-a57c-4996-8243-e5c1dd58cf14"
-					(reference "U15")
+					(reference "U21")
 					(unit 1)
 				)
@@
 		(on_board yes)
 		(dnp no)
-		(property "Reference" "#PWR049"
+		(property "Reference" "#PWR050"
 			(at 133.35 97.79 0)
 			(effects
@@
 			(project "HMI_LVDC-Inverter"
 				(path "/0057333c-5edf-4047-9690-4d1b87a98977/e510606f-6f04-4711-9f2b-d43d4de4a4de/055a40fe-cd38-468e-af40-51b3396e74eb"
+					(reference "#PWR053")
+					(unit 1)
+				)
+				(path "/0057333c-5edf-4047-9690-4d1b87a98977/e510606f-6f04-4711-9f2b-d43d4de4a4de/56ca9b1f-7ac9-4571-b846-7d181a59aeeb"
+					(reference "#PWR051")
+					(unit 1)
+				)
+				(path "/0057333c-5edf-4047-9690-4d1b87a98977/e510606f-6f04-4711-9f2b-d43d4de4a4de/6a364d1f-798c-4d3f-8ad2-c49dde5e0a04"
+					(reference "#PWR055")
+					(unit 1)
+				)
+				(path "/0057333c-5edf-4047-9690-4d1b87a98977/e510606f-6f04-4711-9f2b-d43d4de4a4de/8ed63270-0053-4d5b-bff7-f9f37411008b"
 					(reference "#PWR052")
 					(unit 1)
 				)
-				(path "/0057333c-5edf-4047-9690-4d1b87a98977/e510606f-6f04-4711-9f2b-d43d4de4a4de/56ca9b1f-7ac9-4571-b846-7d181a59aeeb"
+				(path "/0057333c-5edf-4047-9690-4d1b87a98977/e510606f-6f04-4711-9f2b-d43d4de4a4de/bd0135dc-8da7-4e5d-91da-103a4a8ec09c"
 					(reference "#PWR050")
 					(unit 1)
 				)
-				(path "/0057333c-5edf-4047-9690-4d1b87a98977/e510606f-6f04-4711-9f2b-d43d4de4a4de/6a364d1f-798c-4d3f-8ad2-c49dde5e0a04"
+				(path "/0057333c-5edf-4047-9690-4d1b87a98977/e510606f-6f04-4711-9f2b-d43d4de4a4de/d5a41d21-a57c-4996-8243-e5c1dd58cf14"
 					(reference "#PWR054")
 					(unit 1)
 				)
-				(path "/0057333c-5edf-4047-9690-4d1b87a98977/e510606f-6f04-4711-9f2b-d43d4de4a4de/8ed63270-0053-4d5b-bff7-f9f37411008b"
-					(reference "#PWR051")
-					(unit 1)
-				)
-				(path "/0057333c-5edf-4047-9690-4d1b87a98977/e510606f-6f04-4711-9f2b-d43d4de4a4de/bd0135dc-8da7-4e5d-91da-103a4a8ec09c"
-					(reference "#PWR049")
-					(unit 1)
-				)
-				(path "/0057333c-5edf-4047-9690-4d1b87a98977/e510606f-6f04-4711-9f2b-d43d4de4a4de/d5a41d21-a57c-4996-8243-e5c1dd58cf14"
-					(reference "#PWR053")
-					(unit 1)
-				)
