File: Hardware/PCB_Conversor/MedicionCorriente.kicad_sch (KiCad schematic)
At the start: 5 parts, among them U11 ACS712xLCTR-05B

Commit message: Actualizacion conversor
Parts:
- R27: value 150 -> 221
Changed lines of the file:
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@@
 			)
 		)
-		(property "Value" "150"
+		(property "Value" "221"
 			(at 134.62 96.52 90)
 			(effects
