File: Hardware/PCB_Conversor/MedicionTension.kicad_sch (KiCad schematic)
At the start: 10 parts, among them U13 TL431PK, U14 PC817

Commit message: Actualizacion conversor
Parts:
- added R1, R4: 150k, Resistor_SMD:R_0603_1608Metric_Pad0.98x0.95mm_HandSolder, symbol Device:R
- R34: value 470k -> 150k
Connections:
- net Vin_HV: now also R4.1; no longer R34.1
- net at C17.1, R35.1, U13.1 (REF): now also R1.2; no longer R34.2
- new net: R1.1, R34.2
- new net: R34.1, R4.2
Other:
- moved on the sheet: R34, R36
Changed lines of the file:
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@@
+	)
+	(junction
+		(at 116.84 73.66)
+		(diameter 0)
+		(color 0 0 0 0)
 	)
 	(junction
@@
 	)
 	(junction
-		(at 116.84 81.28)
-		(diameter 0)
-		(color 0 0 0 0)
-	)
-	(junction
 		(at 129.54 100.33)
 		(diameter 0)
@@
 	(wire
 		(pts
-			(xy 127 81.28) (xy 129.54 81.28)
+			(xy 127 73.66) (xy 129.54 73.66)
 		)
 		(stroke
@@
 	(wire
 		(pts
-			(xy 116.84 81.28) (xy 119.38 81.28)
+			(xy 116.84 73.66) (xy 119.38 73.66)
 		)
 		(stroke
@@
 	(wire
 		(pts
+			(xy 116.84 73.66) (xy 116.84 74.6625)
+		)
+		(stroke
+			(width 0)
+			(type default)
+		)
+	)
+	(wire
+		(pts
 			(xy 129.54 90.17) (xy 129.54 91.44)
 		)
@@
 	(wire
 		(pts
-			(xy 116.84 81.28) (xy 116.84 86.36)
-		)
-		(stroke
-			(width 0)
-			(type default)
-		)
-	)
-	(wire
-		(pts
 			(xy 116.84 110.49) (xy 129.54 110.49)
 		)
@@
 	(wire
 		(pts
-			(xy 129.54 81.28) (xy 129.54 82.55)
+			(xy 129.54 73.66) (xy 129.54 82.55)
 		)
 		(stroke
@@
 	(wire
 		(pts
-			(xy 116.84 93.98) (xy 116.84 100.33)
+			(xy 116.84 90.17) (xy 116.84 91.44)
 		)
 		(stroke
@@
 	(wire
 		(pts
-			(xy 113.03 81.28) (xy 116.84 81.28)
+			(xy 113.03 73.66) (xy 116.84 73.66)
+		)
+		(stroke
+			(width 0)
+			(type default)
+		)
+	)
+	(wire
+		(pts
+			(xy 116.84 82.2825) (xy 116.84 82.55)
 		)
 		(stroke
@@
 		(pts
 			(xy 152.4 105.41) (xy 156.21 105.41)
+		)
+		(stroke
+			(width 0)
+			(type default)
+		)
+	)
+	(wire
+		(pts
+			(xy 116.84 99.06) (xy 116.84 100.33)
 		)
 		(stroke
@@
 	(hierarchical_label "Vin_HV"
 		(shape input)
-		(at 113.03 81.28 180)
+		(at 113.03 73.66 180)
 		(effects
 			(font
@@
 	(symbol
 		(lib_id "Device:R")
-		(at 123.19 81.28 270)
+		(at 123.19 73.66 270)
 		(unit 1)
 		(exclude_from_sim no)
@@
 		(fields_autoplaced yes)
 		(property "Reference" "R36"
-			(at 123.19 74.93 90)
+			(at 123.19 67.31 90)
 			(effects
 				(font
@@
 		)
 		(property "Value" "220k"
-			(at 123.19 77.47 90)
+			(at 123.19 69.85 90)
 			(effects
 				(font
@@
 		)
 		(property "Footprint" "Resistor_SMD:R_0603_1608Metric_Pad0.98x0.95mm_HandSolder"
-			(at 123.19 79.502 90)
+			(at 123.19 71.882 90)
 			(effects
 				(font
@@
 		)
 		(property "Datasheet" "~"
-			(at 123.19 81.28 0)
+			(at 123.19 73.66 0)
 			(effects
 				(font
@@
 		)
 		(property "Description" "Resistor"
-			(at 123.19 81.28 0)
+			(at 123.19 73.66 0)
 			(effects
 				(font
@@
 				(path "/e60c11d9-ab9e-4760-a4a7-008fcec65a72/c6551446-5e26-4d9a-a5bc-1c867d865e21/6ade7ab7-6233-4c60-8ab6-50f492d9a784"
 					(reference "R43")
+					(unit 1)
+				)
+			)
+		)
+	)
+	(symbol
+		(lib_id "Device:R")
+		(at 116.84 95.25 0)
+		(unit 1)
+		(exclude_from_sim no)
+		(in_bom yes)
+		(on_board yes)
+		(dnp no)
+		(property "Reference" "R1"
+			(at 111.76 94.234 0)
+			(effects
+				(font
+					(size 1.27 1.27)
+				)
+				(justify left)
+			)
+		)
+		(property "Value" "150k"
+			(at 110.744 96.266 0)
+			(effects
+				(font
+					(size 1.27 1.27)
+				)
+				(justify left)
+			)
+		)
+		(property "Footprint" "Resistor_SMD:R_0603_1608Metric_Pad0.98x0.95mm_HandSolder"
+			(at 115.062 95.25 90)
+			(effects
+				(font
+					(size 1.27 1.27)
+				)
+				(hide yes)
+			)
+		)
+		(property "Datasheet" "~"
+			(at 116.84 95.25 0)
+			(effects
+				(font
+					(size 1.27 1.27)
+				)
+				(hide yes)
+			)
+		)
+		(property "Description" "Resistor"
+			(at 116.84 95.25 0)
+			(effects
+				(font
+					(size 1.27 1.27)
+				)
+				(hide yes)
+			)
+		)
+		(pin "1"
+		)
+		(pin "2"
+		)
+		(instances
+			(project "PCB_Conversor"
+				(path "/e60c11d9-ab9e-4760-a4a7-008fcec65a72/c6551446-5e26-4d9a-a5bc-1c867d865e21/0a448165-ee74-4b91-8dde-4d35bebf2843"
+					(reference "R1")
+					(unit 1)
+				)
+				(path "/e60c11d9-ab9e-4760-a4a7-008fcec65a72/c6551446-5e26-4d9a-a5bc-1c867d865e21/6ade7ab7-6233-4c60-8ab6-50f492d9a784"
+					(reference "R3")
 					(unit 1)
 				)
@@
 	(symbol
 		(lib_id "Device:R")
-		(at 116.84 90.17 0)
+		(at 116.84 86.36 0)
 		(unit 1)
 		(exclude_from_sim no)
@@
 		(dnp no)
 		(property "Reference" "R34"
-			(at 111.76 89.154 0)
-			(effects
-				(font
-					(size 1.27 1.27)
-				)
-				(justify left)
-			)
-		)
-		(property "Value" "470k"
-			(at 110.744 91.186 0)
+			(at 111.76 85.344 0)
+			(effects
+				(font
+					(size 1.27 1.27)
+				)
+				(justify left)
+			)
+		)
+		(property "Value" "150k"
+			(at 110.744 87.376 0)
 			(effects
 				(font
@@
 		)
 		(property "Footprint" "Resistor_SMD:R_0603_1608Metric_Pad0.98x0.95mm_HandSolder"
-			(at 115.062 90.17 90)
+			(at 115.062 86.36 90)
 			(effects
 				(font
@@
 		)
 		(property "Datasheet" "~"
-			(at 116.84 90.17 0)
+			(at 116.84 86.36 0)
 			(effects
 				(font
@@
 		)
 		(property "Description" "Resistor"
-			(at 116.84 90.17 0)
+			(at 116.84 86.36 0)
 			(effects
 				(font
@@
 					(unit 1)
 				)
+			)
+		)
+	)
+	(symbol
+		(lib_id "Device:R")
+		(at 116.84 78.4725 0)
+		(unit 1)
+		(exclude_from_sim no)
+		(in_bom yes)
+		(on_board yes)
+		(dnp no)
+		(property "Reference" "R4"
+			(at 111.76 77.4565 0)
+			(effects
+				(font
+					(size 1.27 1.27)
+				)
+				(justify left)
+			)
+		)
+		(property "Value" "150k"
+			(at 110.744 79.4885 0)
+			(effects
+				(font
+					(size 1.27 1.27)
+				)
+				(justify left)
+			)
+		)
+		(property "Footprint" "Resistor_SMD:R_0603_1608Metric_Pad0.98x0.95mm_HandSolder"
+			(at 115.062 78.4725 90)
+			(effects
+				(font
+					(size 1.27 1.27)
+				)
+				(hide yes)
+			)
+		)
+		(property "Datasheet" "~"
+			(at 116.84 78.4725 0)
+			(effects
+				(font
+					(size 1.27 1.27)
+				)
+				(hide yes)
+			)
+		)
+		(property "Description" "Resistor"
+			(at 116.84 78.4725 0)
+			(effects
+				(font
+					(size 1.27 1.27)
+				)
+				(hide yes)
+			)
+		)
+		(pin "1"
+		)
+		(pin "2"
+		)
+		(instances
+			(project "PCB_Conversor"
+				(path "/e60c11d9-ab9e-4760-a4a7-008fcec65a72/c6551446-5e26-4d9a-a5bc-1c867d865e21/0a448165-ee74-4b91-8dde-4d35bebf2843"
+					(reference "R4")
+					(unit 1)
+				)
+				(path "/e60c11d9-ab9e-4760-a4a7-008fcec65a72/c6551446-5e26-4d9a-a5bc-1c867d865e21/6ade7ab7-6233-4c60-8ab6-50f492d9a784"
+					(reference "R5")
+					(unit 1)
+				)
