File: Hardware/PCB_Conversor/PCB_Conversor.kicad_pcb (KiCad board)
At the start: 2 copper layers, 100 x 100 mm, 84 parts, among them Q13 SS8050, Q14 SS8550, Q15 IRFB4110PBF, Q16 SS8050, Q17 SS8550, Q18 IRFB4110PBF, Q19 SS8050, Q20 SS8550, Q21 IRFB4110PBF, Q22 SS8050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

Commit message: Actualizacion conversor
Parts:
- added G***: LOGO, Image:LogoUTN, F.Cu at (128.7, 56.1)
- added G***: LOGO, Image:LogoUTN, F.Cu at (127.7, 77.3)
- added R1: 150k, Resistor_SMD:R_0603_1608Metric_Pad0.98x0.95mm_HandSolder, B.Cu at (105.7, 101.1)
- added R3: 150k, Resistor_SMD:R_0603_1608Metric_Pad0.98x0.95mm_HandSolder, B.Cu at (104.4, 112.6)
- added R4: 150k, Resistor_SMD:R_0603_1608Metric_Pad0.98x0.95mm_HandSolder, B.Cu at (109.0, 101.1)
- added R5: 150k, Resistor_SMD:R_0603_1608Metric_Pad0.98x0.95mm_HandSolder, B.Cu at (111.2, 112.6)
- 12V_PwrCnv1: footprint Connector_Molex:Molex_KK-254_AE-6410-02A_1x02_P2.54mm_Vertical -> Connector_JST:JST_XH_B2B-XH-A_1x02_P2.50mm_Vertical
- HMI_Signal_B1: footprint Connector_Molex:Molex_KK-254_AE-6410-05A_1x05_P2.54mm_Vertical -> Connector_JST:JST_XH_B5B-XH-A_1x05_P2.50mm_Vertical
- R27: value 150 -> 221
- R34, R41: value 470k -> 150k
- moved TP4 14.2 mm to (124.7, 91.9)
- moved R22 2.03 mm to (64.9, 68.4)
- moved R34 1.96 mm to (107.3, 101.1), turned to -90 degrees
- moved R41 1.54 mm to (107.8, 112.6)
- moved C18 1.44 mm to (100.8, 112.1)
- moved 12V_PwrCnv1 0.93 mm to (89.6, 143.4)
- moved TP5 0.89 mm to (124.1, 146.0)
- moved TP6 0.83 mm to (64.9, 90.4)
- moved R24 0.69 mm to (71.3, 91.1)
- moved C17 0.50 mm to (101.5, 101.9)
- moved R38 0.50 mm to (101.5, 103.9)
- moved L1 0.33 mm to (139.4, 106.0)
- moved R44 0.27 mm to (105.8, 114.3)
- moved R43 0.27 mm to (109.4, 114.3)
- moved R45 0.27 mm to (102.2, 114.3)
Connections:
- R34 pad 1: V_HVBus -> Net-(R34-Pad1)
- R34 pad 2: Net-(U13-REF) -> Net-(R1-Pad1)
- R41 pad 1: V_HVBus -> Net-(R41-Pad1)
- R41 pad 2: Net-(U15-REF) -> Net-(R3-Pad1)
Routing:
- net Net-(D5-A): track 52.5 -> 63.2 mm
- net Net-(U15-REF): track 16.8 -> 13.0 mm
- net 12V_Cnv: track 234.6 -> 236.8 mm
- net /Conversor/Modulo conmutador pushpull/Conmutador de potencia/GateInput: track 24.4 -> 26.5 mm
- net Net-(R34-Pad1): track 0.00 -> 1.65 mm
- net Net-(R1-Pad1): track 0.00 -> 1.65 mm
- net Net-(R3-Pad1): track 0.00 -> 1.60 mm
- net Net-(R41-Pad1): track 0.00 -> 1.58 mm
- net Gate_Input_B: track 83.9 -> 82.4 mm
- net GND_Cnv: track 214.1 -> 212.7 mm
- net Net-(U13-REF): track 16.8 -> 16.0 mm
- net Net-(C17-Pad2): track 5.10 -> 4.36 mm
Other:
- outline, holes or cut-outs redrawn
- board text added: "Proyecto Final UTN FRBA Andrenacci, Elian Carra, Lucas"
