File: Hardware/PCB_Inversor/PCB_Inversor.kicad_pcb (KiCad board)
At the start: 2 copper layers, 100 x 76.2 mm, 58 parts, among them Q1 TK8A65D, Q10 SS8050, Q11 SS8050, Q12 SS8050, Q2 TK8A65D, Q3 TK8A65D, Q4 TK8A65D, Q5 TK8A65D, Q6 TK8A65D, Q7 SS8050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

Commit message: Actualizacion Inversor
Parts:
- added G***: LOGO, Image:LogoUTN, F.Cu at (171.3, 104.5)
- 12V_Inv1: footprint Connector_Molex:Molex_KK-254_AE-6410-02A_1x02_P2.54mm_Vertical -> Connector_JST:JST_XH_B2B-XH-A_1x02_P2.50mm_Vertical
- Inv_Signal1, Inv_Signal2: footprint Connector_Molex:Molex_KK-254_AE-6410-04A_1x04_P2.54mm_Vertical -> Connector_JST:JST_XH_B4B-XH-A_1x04_P2.50mm_Vertical
Routing:
- net Net-(12V_Inv1-Pin_1): track 23.1 -> 21.3 mm
Other:
- outline, holes or cut-outs redrawn
- board text added: "Proyecto Final UTN FRBA Andrenacci, Elian Carra, Lucas"
