File: Hardware/PCB_Inversor/inversor.kicad_sch (KiCad schematic)
At the start: 16 parts, among them Q1 TK8A65D, Q2 TK8A65D, Q3 TK8A65D, Q4 TK8A65D, Q5 TK8A65D, Q6 TK8A65D, U1 TMA-12012S-2WR3

Commit message: Actualizacion Inversor
Parts:
- 12V_Inv1: footprint Connector_Molex:Molex_KK-254_AE-6410-02A_1x02_P2.54mm_Vertical -> Connector_JST:JST_XH_B2B-XH-A_1x02_P2.50mm_Vertical
- Inv_Signal1, Inv_Signal2: footprint Connector_Molex:Molex_KK-254_AE-6410-04A_1x04_P2.54mm_Vertical -> Connector_JST:JST_XH_B4B-XH-A_1x04_P2.50mm_Vertical
- Q1, Q2, Q3, Q4, Q5, Q6: value TK8A65D -> STF24N65M2
Changed lines of the file:
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@@
 			)
 		)
-		(property "Footprint" "Connector_Molex:Molex_KK-254_AE-6410-04A_1x04_P2.54mm_Vertical"
+		(property "Footprint" "Connector_JST:JST_XH_B4B-XH-A_1x04_P2.50mm_Vertical"
 			(at 24.13 36.83 0)
 			(effects
@@
 			)
 		)
-		(property "Value" "TK8A65D"
+		(property "Value" "STF24N65M2"
 			(at 113.03 142.2399 0)
 			(effects
@@
 			)
 		)
-		(property "Value" "TK8A65D"
+		(property "Value" "STF24N65M2"
 			(at 173.99 126.9999 0)
 			(effects
@@
 			)
 		)
-		(property "Value" "TK8A65D"
+		(property "Value" "STF24N65M2"
 			(at 143.51 140.9699 0)
 			(effects
@@
 			)
 		)
-		(property "Value" "TK8A65D"
+		(property "Value" "STF24N65M2"
 			(at 173.99 140.9699 0)
 			(effects
@@
 			)
 		)
-		(property "Value" "TK8A65D"
+		(property "Value" "STF24N65M2"
 			(at 113.03 128.2699 0)
 			(effects
@@
 			)
 		)
-		(property "Footprint" "Connector_Molex:Molex_KK-254_AE-6410-04A_1x04_P2.54mm_Vertical"
+		(property "Footprint" "Connector_JST:JST_XH_B4B-XH-A_1x04_P2.50mm_Vertical"
 			(at 24.13 54.61 0)
 			(effects
@@
 			)
 		)
-		(property "Footprint" "Connector_Molex:Molex_KK-254_AE-6410-02A_1x02_P2.54mm_Vertical"
+		(property "Footprint" "Connector_JST:JST_XH_B2B-XH-A_1x02_P2.50mm_Vertical"
 			(at 196.85 81.28 0)
 			(effects
@@
 			)
 		)
-		(property "Value" "TK8A65D"
+		(property "Value" "STF24N65M2"
 			(at 143.51 128.2699 0)
 			(effects
