File: Hardware/PCB_MicroHMI/HMI_LVDC-Inverter.kicad_pcb (KiCad board)
At the start: 2 copper layers, 100 x 90 mm, 117 parts, among them J1 Micro_PwrBus_B1, J10 OLED, J11 Conn_01x06, J2 Screw_Terminal_01x03, J3 Screw_Terminal_01x08, J4 Conn_01x02, J5 Inv_Signal1_A1, J6 Inverter_MEAS, J7 Inv_Signal1, J8 ESP32_Programmer, J9 Inv_Signal2, K2 FINDER-36.11, Q1 BC847, Q2 2N7002, Q3 BC847, Q4 BC847, SW1 SolderJumper_2_Open, U1 STM32F103C8Tx, U10 MCP23017_SO, U11 PC817, U17 PC817, U18 PC817, U19 PC817, U2 ESP32-WROOM-32E-N16, U20 PC817, U21 PC817, U22 PC817, U3 AMS1117-3.3, U4 B1205S-2WR2, U5 AMS1117-3.3, U6 B1205S-2WR2, U7 4N25, U9 PC817, Y1 Crystal 8MHz, Y2 32.768KHz

Commit message: Actualizacion MicroHMI
Routing:
- net +12V_ISO: track 154.5 -> 155.3 mm
Changed lines of the file:
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@@
 			(outputformat 1)
 			(mirror no)
-			(drillshape 1)
+			(drillshape 0)
 			(scaleselection 1)
-			(outputdirectory "")
+			(outputdirectory "GerberFiles/")
 		)
 	)
@@
 	)
 	(segment
-		(start 115.7938 100.066)
-		(end 113.3554 100.066)
-		(width 0.2)
-		(layer "F.Cu")
-		(net 16)
-	)
-	(segment
 		(start 101.7222 95.2372)
 		(end 102.2782 94.6812)
@@
 	)
 	(segment
+		(start 111.7298 99.7548)
+		(end 111.7298 98.4404)
+		(width 0.2)
+		(layer "F.Cu")
+		(net 16)
+	)
+	(segment
 		(start 169.975 94.78)
 		(end 165.725 94.78)
@@
 	)
 	(segment
+		(start 112.041 100.066)
+		(end 111.7298 99.7548)
+		(width 0.2)
+		(layer "F.Cu")
+		(net 16)
+	)
+	(segment
 		(start 107.4518 100.026)
 		(end 107.4626 100.0152)
@@
 	)
 	(segment
-		(start 113.3554 100.066)
-		(end 111.7298 98.4404)
+		(start 115.7938 100.066)
+		(end 112.041 100.066)
 		(width 0.2)
 		(layer "F.Cu")
@@
 	)
 	(segment
-		(start 112.4645 58.1695)
-		(end 111.816 57.521)
-		(width 0.2)
-		(layer "F.Cu")
-		(net 135)
-	)
-	(segment
 		(start 111.816 57.521)
 		(end 112.695 57.521)
@@
 	)
 	(segment
-		(start 112.4645 59.426)
-		(end 112.4645 58.1695)
+		(start 112.425 57.521)
+		(end 111.816 57.521)
 		(width 0.2)
 		(layer "F.Cu")
@@
 		(width 0.2)
 		(layer "F.Cu")
+		(net 135)
+	)
+	(segment
+		(start 112.4645 57.5605)
+		(end 112.425 57.521)
+		(width 0.2)
+		(layer "F.Cu")
+		(net 135)
+	)
+	(segment
+		(start 112.4645 59.426)
+		(end 112.4645 57.5605)
+		(width 0.2)
+		(layer "F.Cu")
