File: Hardware/PCB_MicroHMI/Perifericos.kicad_sch (KiCad schematic)
At the start: 44 parts, among them J10 OLED, J11 Conn_01x06, K2 FINDER-36.11, Q1 BC847, Q2 2N7002, Q3 BC847, Q4 BC847, SW2 SW_MEC_5G, SW3 SW_MEC_5G, SW4 SW_MEC_5G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

Commit message: Actualizacion MicroHMI
Parts:
- R21: value 12 -> 33
Changed lines of the file:
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@@
 			)
 		)
-		(property "Value" "12"
+		(property "Value" "33"
 			(at 145.669 29.972 0)
 			(effects
