File: Hardware/PCB_Integradora/PCB_Integradora.kicad_pcb (KiCad board)
At the start: 2 copper layers, 100 x 100 mm, 40 parts, among them J1 Conn_01x06, J2 USB_OTG, J3 Conn_01x05_Pin, SW1 SW_Push, SW10 SW_MEC_5E, SW2 SW_Push, SW3 SW_Push, SW4 SW_Push, SW5 SW_Push, SW6 SW_Push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

Commit message: Actualizacion placa integradora
Parts:
- moved J2 45.0 mm to (75.4, 71.3), turned to -90 degrees
- moved SW9 37.3 mm to (115.9, 73.8), turned to 180 degrees
- moved SW10 36.7 mm to (115.9, 65.9), turned to 0 degrees
- moved C4 29.8 mm to (83.1, 67.1), turned to 0 degrees
- moved C1 25.0 mm to (109.8, 65.7), turned to 90 degrees
- moved C6 23.9 mm to (109.7, 70.3), turned to -90 degrees
- moved J3 23.9 mm to (87.5, 63.1), turned to -90 degrees
- moved U1 20.5 mm to (87.9, 71.9), turned to -90 degrees
- moved C3 20.0 mm to (105.3, 62.6), turned to 0 degrees
- moved C2 19.2 mm to (91.5, 76.5), turned to 180 degrees
- moved C5 18.9 mm to (105.3, 75.0), turned to 0 degrees
- moved R4 13.4 mm to (95.2, 75.4), turned to 90 degrees
- moved R3 12.4 mm to (97.1, 75.4), turned to 90 degrees
- moved U2 12.3 mm to (104.0, 68.8), turned to 180 degrees
- moved R2 11.3 mm to (96.1, 63.8), turned to 0 degrees
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Other:
- outline, holes or cut-outs redrawn
